File: G030F6_Adaptor.kicad_pcb (KiCad board)
At the start: 2 copper layers, 15.7 x 25.9 mm, 11 parts, among them J1 Conn_01x10, J2 Conn_01x10, J3 SWD, U1 STM32G030F6P6, U2 AP7343D-33W5

Commit message: Track correction, resistor values, updated visualization
Parts:
- D1: value COLOR? -> GREEN
- R1: value ? -> 511R
Changed lines of the file:
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@@
       (effects (font (size 0.9 0.7) (thickness 0.155)))
     )
-    (fp_text value "?" (at 0 1.43 90) (layer "F.Fab")
+    (fp_text value "511R" (at 0 1.43 90) (layer "F.Fab")
       (effects (font (size 1 1) (thickness 0.15)))
     )
@@
       (effects (font (size 0.9 0.7) (thickness 0.155)))
     )
-    (fp_text value "COLOR?" (at 0 1.43 90) (layer "F.Fab")
+    (fp_text value "GREEN" (at 0 1.43 90) (layer "F.Fab")
       (effects (font (size 1 1) (thickness 0.15)))
     )
@@
   )
   (gr_line (start 166.4208 82.1436) (end 166.6748 82.1436) (layer "F.SilkS") (width 0.155))
-  (gr_line (start 157.8864 83.5406) (end 157.734 83.693) (layer "F.SilkS") (width 0.155))
-  (gr_line (start 157.8864 83.5406) (end 157.8864 84.455) (layer "F.SilkS") (width 0.155))
   (gr_rect (start 171.704 98.044) (end 170.4086 99.9236) (layer "F.SilkS") (width 0.15) (fill none))
   (gr_line (start 169.9768 88.5444) (end 170.4848 88.0364) (layer "F.SilkS") (width 0.155))
@@
   (gr_line (start 178.4188 105.313) (end 177.0888 105.313) (layer "F.SilkS") (width 0.12))
   (gr_line (start 177.0888 105.313) (end 177.0888 103.983) (layer "F.SilkS") (width 0.12))
-  (gr_line (start 157.8864 83.5406) (end 158.0388 83.693) (layer "F.SilkS") (width 0.155))
   (gr_line (start 166.4208 82.1436) (end 166.4208 82.3976) (layer "F.SilkS") (width 0.155))
   (gr_line (start 166.751 90.17) (end 168.1988 90.17) (layer "F.SilkS") (width 0.15))
@@
   (via (at 174.498 84.1756) (size 0.6) (drill 0.3) (layers "F.Cu" "B.Cu") (net 2))
   (arc (start 168.1174 93.147) (mid 168.035544 93.163282) (end 167.966151 93.20965) (width 0.35) (layer "F.Cu") (net 2))
-  (segment (start 170.942 83.439) (end 171.706462 83.439) (width 0.35) (layer "F.Cu") (net 3))
-  (segment (start 165.608 81.28) (end 167.767 83.439) (width 0.35) (layer "F.Cu") (net 3))
+  (segment (start 172.908 84.640538) (end 172.048131 83.780669) (width 0.35) (layer "F.Cu") (net 3))
   (segment (start 171.008 85.0955) (end 171.008 83.505) (width 0.35) (layer "F.Cu") (net 3))
+  (segment (start 165.608 81.28) (end 166.545685 82.217685) (width 0.35) (layer "F.Cu") (net 3))
   (segment (start 171.008 83.505) (end 170.942 83.439) (width 0.35) (layer "F.Cu") (net 3))
-  (segment (start 171.706462 83.439) (end 172.908 84.640538) (width 0.35) (layer "F.Cu") (net 3))
   (segment (start 171.008 85.0955) (end 169.7667 85.0955) (width 0.35) (layer "F.Cu") (net 3))
-  (segment (start 172.908 84.640538) (end 172.908 85.0955) (width 0.35) (layer "F.Cu") (net 3))
+  (segment (start 169.4942 83.439) (end 170.942 83.439) (width 0.35) (layer "F.Cu") (net 3))
+  (segment (start 171.22327 83.439) (end 170.942 83.439) (width 0.35) (layer "F.Cu") (net 3))
+  (segment (start 172.908 85.0955) (end 172.908 84.640538) (width 0.35) (layer "F.Cu") (net 3))
   (segment (start 169.7667 85.0955) (end 169.418 84.7468) (width 0.35) (layer "F.Cu") (net 3))
-  (segment (start 167.767 83.439) (end 170.942 83.439) (width 0.35) (layer "F.Cu") (net 3))
+  (arc (start 172.048131 83.780669) (mid 171.669682 83.527797) (end 171.22327 83.439) (width 0.35) (layer "F.Cu") (net 3))
+  (arc (start 166.545685 82.217685) (mid 167.898475 83.121591) (end 169.4942 83.439) (width 0.35) (layer "F.Cu") (net 3))
   (segment (start 169.3495 96.397) (end 168.9314 96.397) (width 0.25) (layer "F.Cu") (net 4))
   (segment (start 165.608 101.6) (end 167.022122 100.185878) (width 0.25) (layer "F.Cu") (net 4))
