File: G030F6_Adaptor.kicad_sch (KiCad schematic)
At the start: 11 parts, among them J1 Conn_01x10, J2 Conn_01x10, J3 SWD, U1 STM32G030F6P6, U2 AP7343D-33W5

Commit message: Track correction, resistor values, updated visualization
Parts:
- D1: value COLOR? -> GREEN
- R1: value ? -> 511R
Other:
- note added: "Headers and pads"
- note added: "LED"
- note added: "Power supply"
- moved on the sheet: D1, J1, J2, J3, R1
